File: input_buffer_bal_XLR_SMD_1206.sch (KiCad schematic (older format))
At the start: 31 parts, among them J1 CH1_XLR, J2 CH2_XLR, J3 POWER, J4 CH1_OUT, J5 CH2_OUT, U1 LM4562, U2 LM4562

Commit message: added project files
Parts:
- C1, C2, C3, C4, C5, C6, C7, C8: footprint local_footprint_lib:C_Disc_D3.8mm_W2.6mm_P2.50mm_centered -> Capacitor_SMD:C_1206_3216Metric
- D1, D2, D3, D4: value P6KE6.8 -> SMF6.0CA; footprint local_footprint_lib:D_DO-15_P12.70mm_Horizontal_centered_TVS -> Diode_SMD:D_SOD-123F
- R1, R10, R2, R3, R4, R5, R6, R7, R8, R9: footprint local_footprint_lib:R_Axial_DIN0207_L6.3mm_D2.5mm_P10.16mm_Horizontal_centered -> Resistor_SMD:R_1206_3216Metric
- U1, U2: footprint local_footprint_lib:DIP-8_W7.62mm_centered -> Package_SO:SOIC-8_3.9x4.9mm_P1.27mm
Changed lines of the file:
@@
 F 0 "R1" V 3793 1500 50  0000 C CNN
 F 1 "100R" V 3884 1500 50  0000 C CNN
-F 2 "local_footprint_lib:R_Axial_DIN0207_L6.3mm_D2.5mm_P10.16mm_Horizontal_centered" V 3930 1500 50  0001 C CNN
+F 2 "Resistor_SMD:R_1206_3216Metric" V 3930 1500 50  0001 C CNN
 F 3 "~" H 4000 1500 50  0001 C CNN
 	1    4000 1500
@@
 U 1 1 642E9979
 P 4000 2500
-F 0 "R2" V 3793 2500 50  0000 C CNN
-F 1 "100R" V 3884 2500 50  0000 C CNN
-F 2 "local_footprint_lib:R_Axial_DIN0207_L6.3mm_D2.5mm_P10.16mm_Horizontal_centered" V 3930 2500 50  0001 C CNN
+F 0 "R2" V 3800 2550 50  0000 C CNN
+F 1 "100R" V 3900 2550 50  0000 C CNN
+F 2 "Resistor_SMD:R_1206_3216Metric" V 3930 2500 50  0001 C CNN
 F 3 "~" H 4000 2500 50  0001 C CNN
 	1    4000 2500
@@
 F 0 "R3" V 3793 3500 50  0000 C CNN
 F 1 "100R" V 3884 3500 50  0000 C CNN
-F 2 "local_footprint_lib:R_Axial_DIN0207_L6.3mm_D2.5mm_P10.16mm_Horizontal_centered" V 3930 3500 50  0001 C CNN
+F 2 "Resistor_SMD:R_1206_3216Metric" V 3930 3500 50  0001 C CNN
 F 3 "~" H 4000 3500 50  0001 C CNN
 	1    4000 3500
@@
 U 1 1 642EA2A0
 P 4000 4500
-F 0 "R4" V 3793 4500 50  0000 C CNN
-F 1 "100R" V 3884 4500 50  0000 C CNN
-F 2 "local_footprint_lib:R_Axial_DIN0207_L6.3mm_D2.5mm_P10.16mm_Horizontal_centered" V 3930 4500 50  0001 C CNN
+F 0 "R4" V 3800 4550 50  0000 C CNN
+F 1 "100R" V 3900 4550 50  0000 C CNN
+F 2 "Resistor_SMD:R_1206_3216Metric" V 3930 4500 50  0001 C CNN
 F 3 "~" H 4000 4500 50  0001 C CNN
 	1    4000 4500
@@
 F 0 "C5" H 4615 1796 50  0000 L CNN
 F 1 "220p" H 4615 1705 50  0000 L CNN
-F 2 "local_footprint_lib:C_Disc_D3.8mm_W2.6mm_P2.50mm_centered" H 4538 1600 50  0001 C CNN
+F 2 "Capacitor_SMD:C_1206_3216Metric" H 4538 1600 50  0001 C CNN
 F 3 "~" H 4500 1750 50  0001 C CNN
 	1    4500 1750
@@
 F 0 "C6" H 4615 2296 50  0000 L CNN
 F 1 "220p" H 4615 2205 50  0000 L CNN
-F 2 "local_footprint_lib:C_Disc_D3.8mm_W2.6mm_P2.50mm_centered" H 4538 2100 50  0001 C CNN
+F 2 "Capacitor_SMD:C_1206_3216Metric" H 4538 2100 50  0001 C CNN
 F 3 "~" H 4500 2250 50  0001 C CNN
 	1    4500 2250
@@
 F 0 "C7" H 4615 3796 50  0000 L CNN
 F 1 "220p" H 4615 3705 50  0000 L CNN
-F 2 "local_footprint_lib:C_Disc_D3.8mm_W2.6mm_P2.50mm_centered" H 4538 3600 50  0001 C CNN
+F 2 "Capacitor_SMD:C_1206_3216Metric" H 4538 3600 50  0001 C CNN
 F 3 "~" H 4500 3750 50  0001 C CNN
 	1    4500 3750
@@
 F 0 "C8" H 4615 4296 50  0000 L CNN
 F 1 "220p" H 4615 4205 50  0000 L CNN
-F 2 "local_footprint_lib:C_Disc_D3.8mm_W2.6mm_P2.50mm_centered" H 4538 4100 50  0001 C CNN
+F 2 "Capacitor_SMD:C_1206_3216Metric" H 4538 4100 50  0001 C CNN
 F 3 "~" H 4500 4250 50  0001 C CNN
 	1    4500 4250
@@
 F 0 "R5" V 4793 2000 50  0000 C CNN
 F 1 "2M2" V 4884 2000 50  0000 C CNN
-F 2 "local_footprint_lib:R_Axial_DIN0207_L6.3mm_D2.5mm_P10.16mm_Horizontal_centered" V 4930 2000 50  0001 C CNN
+F 2 "Resistor_SMD:R_1206_3216Metric" V 4930 2000 50  0001 C CNN
 F 3 "~" H 5000 2000 50  0001 C CNN
 	1    5000 2000
@@
 F 0 "R7" H 5370 1796 50  0000 L CNN
 F 1 "47K" H 5370 1705 50  0000 L CNN
-F 2 "local_footprint_lib:R_Axial_DIN0207_L6.3mm_D2.5mm_P10.16mm_Horizontal_centered" V 5230 1750 50  0001 C CNN
+F 2 "Resistor_SMD:R_1206_3216Metric" V 5230 1750 50  0001 C CNN
 F 3 "~" H 5300 1750 50  0001 C CNN
 	1    5300 1750
@@
 F 0 "R8" H 5370 2296 50  0000 L CNN
 F 1 "47K" H 5370 2205 50  0000 L CNN
-F 2 "local_footprint_lib:R_Axial_DIN0207_L6.3mm_D2.5mm_P10.16mm_Horizontal_centered" V 5230 2250 50  0001 C CNN
+F 2 "Resistor_SMD:R_1206_3216Metric" V 5230 2250 50  0001 C CNN
 F 3 "~" H 5300 2250 50  0001 C CNN
 	1    5300 2250
@@
 F 0 "R6" V 4793 4000 50  0000 C CNN
 F 1 "2M2" V 4884 4000 50  0000 C CNN
-F 2 "local_footprint_lib:R_Axial_DIN0207_L6.3mm_D2.5mm_P10.16mm_Horizontal_centered" V 4930 4000 50  0001 C CNN
+F 2 "Resistor_SMD:R_1206_3216Metric" V 4930 4000 50  0001 C CNN
 F 3 "~" H 5000 4000 50  0001 C CNN
 	1    5000 4000
@@
 F 0 "R9" H 5370 3796 50  0000 L CNN
 F 1 "47K" H 5370 3705 50  0000 L CNN
-F 2 "local_footprint_lib:R_Axial_DIN0207_L6.3mm_D2.5mm_P10.16mm_Horizontal_centered" V 5230 3750 50  0001 C CNN
+F 2 "Resistor_SMD:R_1206_3216Metric" V 5230 3750 50  0001 C CNN
 F 3 "~" H 5300 3750 50  0001 C CNN
 	1    5300 3750
@@
 F 0 "R10" H 5370 4296 50  0000 L CNN
 F 1 "47K" H 5370 4205 50  0000 L CNN
-F 2 "local_footprint_lib:R_Axial_DIN0207_L6.3mm_D2.5mm_P10.16mm_Horizontal_centered" V 5230 4250 50  0001 C CNN
+F 2 "Resistor_SMD:R_1206_3216Metric" V 5230 4250 50  0001 C CNN
 F 3 "~" H 5300 4250 50  0001 C CNN
 	1    5300 4250
@@
 F 0 "U1" H 6200 1967 50  0000 C CNN
 F 1 "LM4562" H 6200 1876 50  0000 C CNN
-F 2 "local_footprint_lib:DIP-8_W7.62mm_centered" H 6200 1600 50  0001 C CNN
+F 2 "Package_SO:SOIC-8_3.9x4.9mm_P1.27mm" H 6200 1600 50  0001 C CNN
 F 3 "http://www.ti.com/lit/ds/symlink/lm4562.pdf" H 6200 1600 50  0001 C CNN
 	1    6200 1600
@@
 F 0 "U1" H 6200 2967 50  0000 C CNN
 F 1 "LM4562" H 6200 2876 50  0000 C CNN
-F 2 "local_footprint_lib:DIP-8_W7.62mm_centered" H 6200 2600 50  0001 C CNN
+F 2 "Package_SO:SOIC-8_3.9x4.9mm_P1.27mm" H 6200 2600 50  0001 C CNN
 F 3 "http://www.ti.com/lit/ds/symlink/lm4562.pdf" H 6200 2600 50  0001 C CNN
 	2    6200 2600
@@
 F 0 "U1" H 2508 6146 50  0000 L CNN
 F 1 "LM4562" H 2508 6055 50  0000 L CNN
-F 2 "local_footprint_lib:DIP-8_W7.62mm_centered" H 2550 6100 50  0001 C CNN
+F 2 "Package_SO:SOIC-8_3.9x4.9mm_P1.27mm" H 2550 6100 50  0001 C CNN
 F 3 "http://www.ti.com/lit/ds/symlink/lm4562.pdf" H 2550 6100 50  0001 C CNN
 	3    2550 6100
@@
 F 0 "U2" H 6200 3967 50  0000 C CNN
 F 1 "LM4562" H 6200 3876 50  0000 C CNN
-F 2 "local_footprint_lib:DIP-8_W7.62mm_centered" H 6200 3600 50  0001 C CNN
+F 2 "Package_SO:SOIC-8_3.9x4.9mm_P1.27mm" H 6200 3600 50  0001 C CNN
 F 3 "http://www.ti.com/lit/ds/symlink/lm4562.pdf" H 6200 3600 50  0001 C CNN
 	1    6200 3600
@@
 F 0 "U2" H 6200 4967 50  0000 C CNN
 F 1 "LM4562" H 6200 4876 50  0000 C CNN
-F 2 "local_footprint_lib:DIP-8_W7.62mm_centered" H 6200 4600 50  0001 C CNN
+F 2 "Package_SO:SOIC-8_3.9x4.9mm_P1.27mm" H 6200 4600 50  0001 C CNN
 F 3 "http://www.ti.com/lit/ds/symlink/lm4562.pdf" H 6200 4600 50  0001 C CNN
 	2    6200 4600
@@
 F 0 "U2" H 3008 6146 50  0000 L CNN
 F 1 "LM4562" H 3008 6055 50  0000 L CNN
-F 2 "local_footprint_lib:DIP-8_W7.62mm_centered" H 3050 6100 50  0001 C CNN
+F 2 "Package_SO:SOIC-8_3.9x4.9mm_P1.27mm" H 3050 6100 50  0001 C CNN
 F 3 "http://www.ti.com/lit/ds/symlink/lm4562.pdf" H 3050 6100 50  0001 C CNN
 	3    3050 6100
@@
 F 0 "C3" H 3565 6296 50  0000 L CNN
 F 1 "100n" H 3565 6205 50  0000 L CNN
-F 2 "local_footprint_lib:C_Disc_D3.8mm_W2.6mm_P2.50mm_centered" H 3488 6100 50  0001 C CNN
+F 2 "Capacitor_SMD:C_1206_3216Metric" H 3488 6100 50  0001 C CNN
 F 3 "~" H 3450 6250 50  0001 C CNN
 	1    3450 6250
@@
 F 0 "C4" H 4015 6296 50  0000 L CNN
 F 1 "100n" H 4015 6205 50  0000 L CNN
-F 2 "local_footprint_lib:C_Disc_D3.8mm_W2.6mm_P2.50mm_centered" H 3938 6100 50  0001 C CNN
+F 2 "Capacitor_SMD:C_1206_3216Metric" H 3938 6100 50  0001 C CNN
 F 3 "~" H 3900 6250 50  0001 C CNN
 	1    3900 6250
@@
 F 0 "C1" H 1715 5996 50  0000 L CNN
 F 1 "100n" H 1715 5905 50  0000 L CNN
-F 2 "local_footprint_lib:C_Disc_D3.8mm_W2.6mm_P2.50mm_centered" H 1638 5800 50  0001 C CNN
+F 2 "Capacitor_SMD:C_1206_3216Metric" H 1638 5800 50  0001 C CNN
 F 3 "~" H 1600 5950 50  0001 C CNN
 	1    1600 5950
@@
 F 0 "C2" H 2165 5996 50  0000 L CNN
 F 1 "100n" H 2165 5905 50  0000 L CNN
-F 2 "local_footprint_lib:C_Disc_D3.8mm_W2.6mm_P2.50mm_centered" H 2088 5800 50  0001 C CNN
+F 2 "Capacitor_SMD:C_1206_3216Metric" H 2088 5800 50  0001 C CNN
 F 3 "~" H 2050 5950 50  0001 C CNN
 	1    2050 5950
@@
 P 3500 1750
 F 0 "D1" V 3454 1830 50  0000 L CNN
-F 1 "P6KE6.8" V 3545 1830 50  0000 L CNN
-F 2 "local_footprint_lib:D_DO-15_P12.70mm_Horizontal_centered_TVS" H 3500 1750 50  0001 C CNN
+F 1 "SMF6.0CA" V 3545 1830 50  0000 L CNN
+F 2 "Diode_SMD:D_SOD-123F" H 3500 1750 50  0001 C CNN
 F 3 "~" H 3500 1750 50  0001 C CNN
 	1    3500 1750
@@
 P 3500 2250
 F 0 "D2" V 3454 2330 50  0000 L CNN
-F 1 "P6KE6.8" V 3545 2330 50  0000 L CNN
-F 2 "local_footprint_lib:D_DO-15_P12.70mm_Horizontal_centered_TVS" H 3500 2250 50  0001 C CNN
+F 1 "SMF6.0CA" V 3545 2330 50  0000 L CNN
+F 2 "Diode_SMD:D_SOD-123F" H 3500 2250 50  0001 C CNN
 F 3 "~" H 3500 2250 50  0001 C CNN
 	1    3500 2250
@@
 P 3500 3750
 F 0 "D3" V 3454 3830 50  0000 L CNN
-F 1 "P6KE6.8" V 3545 3830 50  0000 L CNN
-F 2 "local_footprint_lib:D_DO-15_P12.70mm_Horizontal_centered_TVS" H 3500 3750 50  0001 C CNN
+F 1 "SMF6.0CA" V 3545 3830 50  0000 L CNN
+F 2 "Diode_SMD:D_SOD-123F" H 3500 3750 50  0001 C CNN
 F 3 "~" H 3500 3750 50  0001 C CNN
 	1    3500 3750
@@
 P 3500 4250
 F 0 "D4" V 3454 4330 50  0000 L CNN
-F 1 "P6KE6.8" V 3545 4330 50  0000 L CNN
-F 2 "local_footprint_lib:D_DO-15_P12.70mm_Horizontal_centered_TVS" H 3500 4250 50  0001 C CNN
+F 1 "SMF6.0CA" V 3545 4330 50  0000 L CNN
+F 2 "Diode_SMD:D_SOD-123F" H 3500 4250 50  0001 C CNN
 F 3 "~" H 3500 4250 50  0001 C CNN
 	1    3500 4250

Commit message: rev1.1 fixes major issues with the pcb layout
Parts:
- C1, C2, C3, C4, C5, C6, C7, C8: footprint Capacitor_SMD:C_1206_3216Metric -> Capacitor_SMD:C_1206_3216Metric_Pad1.42x1.75mm_HandSolder
Changed lines of the file:
@@
 F 0 "C5" H 4615 1796 50  0000 L CNN
 F 1 "220p" H 4615 1705 50  0000 L CNN
-F 2 "Capacitor_SMD:C_1206_3216Metric" H 4538 1600 50  0001 C CNN
+F 2 "Capacitor_SMD:C_1206_3216Metric_Pad1.42x1.75mm_HandSolder" H 4538 1600 50  0001 C CNN
 F 3 "~" H 4500 1750 50  0001 C CNN
 	1    4500 1750
@@
 F 0 "C6" H 4615 2296 50  0000 L CNN
 F 1 "220p" H 4615 2205 50  0000 L CNN
-F 2 "Capacitor_SMD:C_1206_3216Metric" H 4538 2100 50  0001 C CNN
+F 2 "Capacitor_SMD:C_1206_3216Metric_Pad1.42x1.75mm_HandSolder" H 4538 2100 50  0001 C CNN
 F 3 "~" H 4500 2250 50  0001 C CNN
 	1    4500 2250
@@
 F 0 "C7" H 4615 3796 50  0000 L CNN
 F 1 "220p" H 4615 3705 50  0000 L CNN
-F 2 "Capacitor_SMD:C_1206_3216Metric" H 4538 3600 50  0001 C CNN
+F 2 "Capacitor_SMD:C_1206_3216Metric_Pad1.42x1.75mm_HandSolder" H 4538 3600 50  0001 C CNN
 F 3 "~" H 4500 3750 50  0001 C CNN
 	1    4500 3750
@@
 F 0 "C8" H 4615 4296 50  0000 L CNN
 F 1 "220p" H 4615 4205 50  0000 L CNN
-F 2 "Capacitor_SMD:C_1206_3216Metric" H 4538 4100 50  0001 C CNN
+F 2 "Capacitor_SMD:C_1206_3216Metric_Pad1.42x1.75mm_HandSolder" H 4538 4100 50  0001 C CNN
 F 3 "~" H 4500 4250 50  0001 C CNN
 	1    4500 4250
@@
 F 0 "C3" H 3565 6296 50  0000 L CNN
 F 1 "100n" H 3565 6205 50  0000 L CNN
-F 2 "Capacitor_SMD:C_1206_3216Metric" H 3488 6100 50  0001 C CNN
+F 2 "Capacitor_SMD:C_1206_3216Metric_Pad1.42x1.75mm_HandSolder" H 3488 6100 50  0001 C CNN
 F 3 "~" H 3450 6250 50  0001 C CNN
 	1    3450 6250
@@
 F 0 "C4" H 4015 6296 50  0000 L CNN
 F 1 "100n" H 4015 6205 50  0000 L CNN
-F 2 "Capacitor_SMD:C_1206_3216Metric" H 3938 6100 50  0001 C CNN
+F 2 "Capacitor_SMD:C_1206_3216Metric_Pad1.42x1.75mm_HandSolder" H 3938 6100 50  0001 C CNN
 F 3 "~" H 3900 6250 50  0001 C CNN
 	1    3900 6250
@@
 F 0 "C1" H 1715 5996 50  0000 L CNN
 F 1 "100n" H 1715 5905 50  0000 L CNN
-F 2 "Capacitor_SMD:C_1206_3216Metric" H 1638 5800 50  0001 C CNN
+F 2 "Capacitor_SMD:C_1206_3216Metric_Pad1.42x1.75mm_HandSolder" H 1638 5800 50  0001 C CNN
 F 3 "~" H 1600 5950 50  0001 C CNN
 	1    1600 5950
@@
 F 0 "C2" H 2165 5996 50  0000 L CNN
 F 1 "100n" H 2165 5905 50  0000 L CNN
-F 2 "Capacitor_SMD:C_1206_3216Metric" H 2088 5800 50  0001 C CNN
+F 2 "Capacitor_SMD:C_1206_3216Metric_Pad1.42x1.75mm_HandSolder" H 2088 5800 50  0001 C CNN
 F 3 "~" H 2050 5950 50  0001 C CNN
 	1    2050 5950

Commit message: rev1.2 changed power connector
Parts:
- removed J3: POWER, local_footprint_lib:TerminalBlock_ Amphenol_01_03_P3.50mm, symbol Connector:Conn_01x03_Male
- added J3: POWER, local_footprint_lib:TerminalBlock_ Amphenol_01_02_P3.50mm, symbol Connector:Screw_Terminal_01x02
Connections:
- wire segments 112 -> 110
Changed lines of the file:
@@
-$EndComp
-$Comp
-L Connector:Conn_01x03_Male J3
-U 1 1 64303384
-P 5150 6100
-F 0 "J3" H 5122 6032 50  0000 R CNN
-F 1 "POWER" H 5122 6123 50  0000 R CNN
-F 2 "local_footprint_lib:TerminalBlock_ Amphenol_01_03_P3.50mm" H 5150 6100 50  0001 C CNN
-F 3 "~" H 5150 6100 50  0001 C CNN
-	1    5150 6100
-	-1   0    0    1
 $EndComp
 $Comp
@@
 L power:+15V #PWR010
 U 1 1 64419D7E
-P 4800 5900
-F 0 "#PWR010" H 4800 5750 50  0001 C CNN
-F 1 "+15V" H 4815 6073 50  0000 C CNN
-F 2 "" H 4800 5900 50  0001 C CNN
-F 3 "" H 4800 5900 50  0001 C CNN
-	1    4800 5900
-	1    0    0    -1
-$EndComp
-$Comp
-L power:GND #PWR09
-U 1 1 6441BDA0
-P 4550 5900
-F 0 "#PWR09" H 4550 5650 50  0001 C CNN
-F 1 "GND" H 4555 5727 50  0000 C CNN
-F 2 "" H 4550 5900 50  0001 C CNN
-F 3 "" H 4550 5900 50  0001 C CNN
-	1    4550 5900
-	-1   0    0    1
-$EndComp
-Wire Wire Line
-	4800 5900 4800 6000
-Wire Wire Line
-	4800 6000 4950 6000
-Wire Wire Line
-	4950 6100 4550 6100
-Wire Wire Line
-	4550 6100 4550 5900
+P 4800 6000
+F 0 "#PWR010" H 4800 5850 50  0001 C CNN
+F 1 "+15V" H 4815 6173 50  0000 C CNN
+F 2 "" H 4800 6000 50  0001 C CNN
+F 3 "" H 4800 6000 50  0001 C CNN
+	1    4800 6000
+	1    0    0    -1
+$EndComp
+Wire Wire Line
+	4800 6000 4800 6100
+Wire Wire Line
+	4800 6100 4950 6100
 Wire Wire Line
 	4950 6200 4850 6200
@@
 	1    0    0    -1
 $EndComp
+$Comp
+L Connector:Screw_Terminal_01x02 J3
+U 1 1 64795BCC
+P 5150 6100
+F 0 "J3" H 5230 6092 50  0000 L CNN
+F 1 "POWER" H 5230 6001 50  0000 L CNN
+F 2 "local_footprint_lib:TerminalBlock_ Amphenol_01_02_P3.50mm" H 5150 6100 50  0001 C CNN
+F 3 "~" H 5150 6100 50  0001 C CNN
+	1    5150 6100
+	1    0    0    -1
+$EndComp

Commit message: revised with added option to change gain
Parts:
- removed C7, C8: 220p, Capacitor_SMD:C_1206_3216Metric_Pad1.42x1.75mm_HandSolder, symbol Device:C
- removed D1, D2, D3, D4: SMF6.0CA, Diode_SMD:D_SOD-123F, symbol Device:D_TVS
- added C5, C6: 1n, Capacitor_SMD:C_1206_3216Metric_Pad1.42x1.75mm_HandSolder, symbol Device:C
- added J6, J7: CH1_OUT, local_footprint_lib:TerminalBlock_ Amphenol_01_03_P3.50mm, symbol Connector:Screw_Terminal_01x03
- added R11, R12, R13, R14: 1K, Resistor_SMD:R_1206_3216Metric, symbol Device:R
- added R15, R16: 1K3, Resistor_SMD:R_1206_3216Metric, symbol Device:R
- added R17, R18: 3k, Resistor_SMD:R_1206_3216Metric, symbol Device:R
- C3: renamed from C5; value 220p -> 1n
- C4: renamed from C6; value 220p -> 1n
- J4: value CH1_OUT -> Gain; footprint local_footprint_lib:TerminalBlock_ Amphenol_01_03_P3.50mm -> Connector_PinHeader_2.54mm:PinHeader_1x03_P2.54mm_Vertical
- J5: value CH2_OUT -> Gain; footprint local_footprint_lib:TerminalBlock_ Amphenol_01_03_P3.50mm -> Connector_PinHeader_2.54mm:PinHeader_1x03_P2.54mm_Vertical
- renumbered C3 to C7, C4 to C8
Connections:
- wire segments 110 -> 114
Other:
- moved on the sheet: C1, C2, C3, C4, C7, C8, J1, J3, R1, R2, R5, R7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

Commit message: initial commit
Parts:
- added SW? (x2): SW_SP3T, symbol Switch:SW_SP3T
- added SW?: SW_4PDT, symbol Switch:SW_4PDT
Other:
- moved on the sheet: C1, C2, C3, C4, C5, C6, C7, C8, J1, J2, J3, J4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

Commit message: initial commit
Parts:
- removed J5: Gain, Connector_PinHeader_2.54mm:PinHeader_1x03_P2.54mm_Vertical, symbol Connector:Conn_01x03_Male
- removed J7: CH1_OUT, local_footprint_lib:TerminalBlock_ Amphenol_01_03_P3.50mm, symbol Connector:Screw_Terminal_01x03
- removed SW?: SW_SP3T, symbol Switch:SW_SP3T
- added J6: CH1_OUT, local_footprint_lib:TerminalBlock_ Amphenol_01_03_P3.50mm, symbol Connector:Screw_Terminal_01x03
- added SW3: GAIN_CH2, symbol Switch:SW_SP3T
- R15: value 1K3 -> 1K
- R16: value 1K3 -> 560R
- R17: value 3k -> 1K
- R18: value 3k -> 560R
- SW1: renamed from SW?; value SW_4PDT -> BTL
- SW2: renamed from SW?; value SW_SP3T -> GAIN_CH1
- renumbered C7 to C3, C8 to C4, C3 to C5, C4 to C6, C5 to C7, C6 to C8, J3 to J1, J1 to J2, J2 to J3, J6 to J5
Connections:
- net GND: now also SW1.10 (A), SW1.7 (A), J6.3 (Pin_3)
- net at R2.2: now also SW1.8 (B); no longer J2.3
- net at J5.2 (Pin_2), R11.1, U1.1: now also SW2.3; no longer J4.2 (Pin_2)
- net at J5.1 (Pin_1), R12.1, U1.7: now also R15.1, R16.1; no longer R15.2, R17.2
- net at J4.1 (Pin_1): no longer R17.1
- net at J4.3 (Pin_3): no longer R15.1
- net at R3.2: now also SW1.5 (B); no longer J3.2
- net at R4.2: now also SW1.11 (B); no longer J3.3
- net at R13.1, U2.1: now also J6.2 (Pin_2), SW3.3
- net at R14.1, U2.7: now also R17.1, R18.1, J6.1 (Pin_1); no longer R16.2, R18.2
- net at SW2.2: now also R15.2
- net at SW2.4: now also R16.2
- net at SW1.1 (A): now also SW1.4 (A)
- net at SW1.12 (C): now also J3.3
- net at SW1.2 (B): now also J2.3
- net at SW1.3 (C): now also SW1.9 (C)
- net at SW1.6 (C): now also J3.2
- new net: R17.2, SW3.2
- new net: R18.2, SW3.4
- no-connect marks 0 -> 2
Other:
- moved on the sheet: C5, C6, C7, C8, J4, J5, R1, R10, R11, R12, R13, R14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

Commit message: initial commit
Parts:
- removed J4: Gain, Connector_PinHeader_2.54mm:PinHeader_1x03_P2.54mm_Vertical, symbol Connector:Conn_01x03_Male
- removed SW2: GAIN_CH1, symbol Switch:SW_SP3T
- removed SW3: GAIN_CH2, symbol Switch:SW_SP3T
- added SW2: GAIN_CH1, symbol Switch:SW_DIP_x02
- added SW3: GAIN_CH2, symbol Switch:SW_DIP_x02
- R15, R17: value 1K -> 3K3
- R16, R18: value 560R -> 910R
Connections:
- net at J5.2 (Pin_2), R11.1, U1.1: now also SW2.1, SW2.2
- net at J6.2 (Pin_2), R13.1, U2.1: now also SW3.1, SW3.2
- net at R15.2: now also SW2.4
- net at R16.2: now also SW2.3
- net at R17.2: now also SW3.4
- net at R18.2: now also SW3.3
- no-connect marks 2 -> 0
Other:
- moved on the sheet: C1, C2, C3, C4, H1, H2, J1, R15, R16, U1C, U2C

Commit message: footprints updates
Parts:
- SW1: footprint (none) -> local_footprint_lib:SW_SS-42H11_4PDT
- SW2, SW3: footprint (none) -> local_footprint_lib:SW_DIP_SPSTx02_Slide_W7.62mm_P2.54mm
Connections:
- net GND: now also J6.1 (Pin_1), SW1.13 (GND); no longer J6.3 (Pin_3)
- net at C7.1, R3.1, R9.1: now also U2.5 (+); no longer U2.3 (+)
- net at C8.2, R10.2, R4.1: now also U2.3 (+); no longer U2.5 (+)
- net at J6.2 (Pin_2), R13.1, SW3.1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: now also U2.7; no longer U2.1
- net at U2.2 (-): now also R14.2; no longer R13.2
- net at U2.6 (-): now also R13.2; no longer R14.2
- net at R14.1, R17.1, R18.1: now also J6.3 (Pin_3), U2.1; no longer J6.1 (Pin_1), U2.7
Other:
- moved on the sheet: U2A, U2B
Changed lines of the file:
@@
 encoding utf-8
 Sheet 1 1
-Title "Balanced input impedance matshin buffer with XRL connectors"
-Date "2023-04-06"
+Title "Balanced input buffer with XRL connectors"
+Date "2024-01-18"
 Rev "R1.0"
-Comp "Bilous Sound"
+Comp "Pavlo's Lab"
 Comment1 ""
 Comment2 ""
@@
 L Amplifier_Operational:LM4562 U2
 U 1 1 65A8727D
+P 5250 6100
+F 0 "U2" H 5250 6467 50  0000 C CNN
+F 1 "LM4562" H 5250 6376 50  0000 C CNN
+F 2 "Package_SO:SOIC-8_3.9x4.9mm_P1.27mm" H 5250 6100 50  0001 C CNN
+F 3 "http://www.ti.com/lit/ds/symlink/lm4562.pdf" H 5250 6100 50  0001 C CNN
+	1    5250 6100
+	1    0    0    1
+$EndComp
+$Comp
+L Amplifier_Operational:LM4562 U2
+U 2 1 65A87283
 P 5250 4900
 F 0 "U2" H 5250 5267 50  0000 C CNN
@@
 F 2 "Package_SO:SOIC-8_3.9x4.9mm_P1.27mm" H 5250 4900 50  0001 C CNN
 F 3 "http://www.ti.com/lit/ds/symlink/lm4562.pdf" H 5250 4900 50  0001 C CNN
-	1    5250 4900
-	1    0    0    -1
-$EndComp
-$Comp
-L Amplifier_Operational:LM4562 U2
-U 2 1 65A87283
-P 5250 6100
-F 0 "U2" H 5250 6467 50  0000 C CNN
-F 1 "LM4562" H 5250 6376 50  0000 C CNN
-F 2 "Package_SO:SOIC-8_3.9x4.9mm_P1.27mm" H 5250 6100 50  0001 C CNN
-F 3 "http://www.ti.com/lit/ds/symlink/lm4562.pdf" H 5250 6100 50  0001 C CNN
-	2    5250 6100
-	1    0    0    1
+	2    5250 4900
+	1    0    0    -1
 $EndComp
 $Comp
@@
 F 0 "SW1" H 2275 4681 50  0000 C CNN
 F 1 "BTL" H 2275 4590 50  0000 C CNN
-F 2 "" H 2220 4000 50  0001 C CNN
+F 2 "local_footprint_lib:SW_SS-42H11_4PDT" H 2220 4000 50  0001 C CNN
 F 3 "~" H 2220 4000 50  0001 C CNN
 	1    2300 3850
@@
 Wire Wire Line
 	2550 4250 2450 4250
-Wire Wire Line
-	2100 4350 2000 4350
-Wire Wire Line
-	2000 4350 2000 6000
-Wire Wire Line
-	2000 6000 3000 6000
 Wire Wire Line
 	3000 5000 1850 5000
@@
 F 3 "~" H 7400 5500 50  0001 C CNN
 	1    7400 5500
-	1    0    0    1
+	1    0    0    -1
 $EndComp
 Wire Wire Line
@@
 F 0 "SW2" H 5950 2267 50  0000 C CNN
 F 1 "GAIN_CH1" H 5950 2176 50  0000 C CNN
-F 2 "" H 5950 1900 50  0001 C CNN
+F 2 "local_footprint_lib:SW_DIP_SPSTx02_Slide_W7.62mm_P2.54mm" H 5950 1900 50  0001 C CNN
 F 3 "~" H 5950 1900 50  0001 C CNN
 	1    5950 1900
@@
 F 0 "SW3" H 5950 5767 50  0000 C CNN
 F 1 "GAIN_CH2" H 5950 5676 50  0000 C CNN
-F 2 "" H 5950 5400 50  0001 C CNN
+F 2 "local_footprint_lib:SW_DIP_SPSTx02_Slide_W7.62mm_P2.54mm" H 5950 5400 50  0001 C CNN
 F 3 "~" H 5950 5400 50  0001 C CNN
 	1    5950 5400
@@
 Connection ~ 5550 5300
 Connection ~ 5650 5300
+$Comp
+L power:GND #PWR0101
+U 1 1 65AE8933
+P 2050 4550
+F 0 "#PWR0101" H 2050 4300 50  0001 C CNN
+F 1 "GND" H 2055 4377 50  0001 C CNN
+F 2 "" H 2050 4550 50  0001 C CNN
+F 3 "" H 2050 4550 50  0001 C CNN
+	1    2050 4550
+	1    0    0    -1
+$EndComp
+Wire Wire Line
+	2100 4500 2050 4500
+Wire Wire Line
+	2050 4500 2050 4550
+Wire Wire Line
+	1950 4350 1950 6000
+Wire Wire Line
+	1950 4350 2100 4350
+Wire Wire Line
+	1950 6000 3000 6000
+Connection ~ 5550 4900
+Connection ~ 5550 6100
 $EndSCHEMATC
