File: input_buffer_bal_XLR_SMD_1206.sch (KiCad schematic (older format))
At the start: 38 parts, among them J1 POWER, J2 CH1_XLR, J3 CH2_XLR, J5 CH1_OUT, J6 CH1_OUT, SW1 BTL, SW2 GAIN_CH1, SW3 GAIN_CH2, U1 LM4562, U2 LM4562

Commit message: finished layout
Connections:
- net GND: now also J5.1 (Pin_1), J6.3 (Pin_3); no longer J5.3 (Pin_3), J6.1 (Pin_1)
- net at J5.2 (Pin_2), R11.1, U1.1: no longer SW2.1, SW2.2
- net at R11.2, U1.2 (-): now also SW2.1, SW2.2
- net at R12.2, U1.6 (-): now also R15.1, R16.1
- net at R14.2, U2.2 (-): now also R17.1, R18.1
- net at R13.2, U2.6 (-): now also SW3.1, SW3.2
- net at J6.2 (Pin_2), R13.1, U2.7: no longer SW3.1, SW3.2
- new net: J5.3 (Pin_3), R12.1, U1.7
- new net: J6.1 (Pin_1), R14.1, U2.1
Other:
- moved on the sheet: R11, R12, R13, R14, R15, R16, R17, R18, SW2, SW3, U1A, U1B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
