File: input_buffer_bal_XLR_SMD_1206.kicad_pcb (KiCad board)
At the start: 2 copper layers, 70 x 54.8 mm, 37 parts, among them J1 CH1_XLR, J2 CH2_XLR, J3 POWER, J4 Gain, J5 Gain, J6 CH1_OUT, J7 CH1_OUT, U1 LM4562, U2 LM4562

Commit message: footprints updates
Parts:
- removed J4: Gain, Connector_PinHeader_2.54mm:PinHeader_1x03_P2.54mm_Vertical
- removed the J5 at (140.0, 110.8)
- removed J7: CH1_OUT, local_footprint_lib:TerminalBlock_ Amphenol_01_03_P3.50mm
- added J6: CH1_OUT, local_footprint_lib:TerminalBlock_ Amphenol_01_03_P3.50mm, F.Cu at (156.2, 105.0)
- added SW1: BTL, local_footprint_lib:SW_SS-42H11_4PDT, F.Cu at (125.0, 135.0)
- added SW2: GAIN_CH1, local_footprint_lib:SW_DIP_SPSTx02_Slide_W7.62mm_P2.54mm, F.Cu at (106.2, 108.8)
- added SW3: GAIN_CH2, local_footprint_lib:SW_DIP_SPSTx02_Slide_W7.62mm_P2.54mm, F.Cu at (143.8, 108.8)
- R15: value 1K3 -> 3K3
- R16: value 1K3 -> 910R
- R17: value 3k -> 3K3
- R18: value 3k -> 910R
- moved R16 47.8 mm to (98.2, 114.2)
- moved R17 45.9 mm to (151.8, 114.2), turned to 180 degrees
- moved C7 31.5 mm to (168.2, 123.2), turned to 0 degrees
- moved R13 31.5 mm to (168.2, 120.2), turned to 0 degrees
- moved R3 31.5 mm to (168.2, 126.2), turned to 0 degrees
- moved R9 21.5 mm to (163.2, 131.2)
- moved C1 15.0 mm to (91.0, 115.8)
- moved C2 15.0 mm to (161.0, 115.8)
- moved C3 15.0 mm to (89.0, 125.8)
- moved C4 15.0 mm to (159.0, 125.8)
- moved C5 15.0 mm to (81.8, 123.2)
- moved C6 15.0 mm to (98.2, 123.2)
- moved R1 15.0 mm to (81.8, 126.2)
- moved R11 15.0 mm to (81.8, 120.2)
- moved R12 15.0 mm to (98.2, 120.2)
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- renumbered C7 to C3, C8 to C4, C3 to C5, C4 to C6, C5 to C7, C6 to C8, J3 to J1, J1 to J2, J2 to J3, J6 to J5
Connections:
- C7 pad 1: Net-(C5-Pad1) (its old number) -> Net-(C7-Pad1)
- C8 pad 2: Net-(C6-Pad2) (its old number) -> Net-(C8-Pad2)
- J2 pad 3: Net-(J1-Pad3) -> Net-(J2-Pad3)
- J3 pad 2: Net-(J2-Pad2) (its old number) -> Net-(J3-Pad2)
- J3 pad 3: Net-(J2-Pad3) -> Net-(J3-Pad3)
- J5 pad 1: Net-(J6-Pad1) -> Net-(J5-Pad1)
- R10 pad 2: Net-(C6-Pad2) (its old number) -> Net-(C8-Pad2)
- R12 pad 1: Net-(J6-Pad1) -> Net-(J5-Pad1)
- R13 pad 1: Net-(J5-Pad2) (its old number) -> Net-(J6-Pad2)
- R14 pad 1: Net-(J7-Pad1) -> Net-(J6-Pad3)
- R15 pad 1: Net-(J4-Pad3) -> Net-(J5-Pad1)
- R15 pad 2: Net-(J6-Pad1) -> Net-(R15-Pad2)
- R16 pad 1: Net-(J5-Pad3) -> Net-(J5-Pad1)
- R16 pad 2: Net-(J7-Pad1) -> Net-(R16-Pad2)
- R17 pad 1: Net-(J4-Pad1) -> Net-(J6-Pad3)
- R17 pad 2: Net-(J6-Pad1) -> Net-(R17-Pad2)
- R18 pad 1: Net-(J5-Pad1) -> Net-(J6-Pad3)
- R18 pad 2: Net-(J7-Pad1) -> Net-(R18-Pad2)
- R2 pad 2: Net-(J1-Pad3) -> Net-(R2-Pad2)
- R3 pad 1: Net-(C5-Pad1) (its old number) -> Net-(C7-Pad1)
- R3 pad 2: Net-(J2-Pad2) (its old number) -> Net-(R3-Pad2)
- R4 pad 1: Net-(C6-Pad2) (its old number) -> Net-(C8-Pad2)
- R4 pad 2: Net-(J2-Pad3) -> Net-(R4-Pad2)
- R9 pad 1: Net-(C5-Pad1) (its old number) -> Net-(C7-Pad1)
- U1 pad 7: Net-(J6-Pad1) -> Net-(J5-Pad1)
- U2 pad 1: Net-(J5-Pad2) (its old number) -> Net-(J6-Pad3)
- U2 pad 2: Net-(R13-Pad2) -> Net-(R14-Pad2)
- U2 pad 3: Net-(C5-Pad1) (its old number) -> Net-(C8-Pad2)
- U2 pad 5: Net-(C6-Pad2) (its old number) -> Net-(C7-Pad1)
- U2 pad 6: Net-(R14-Pad2) -> Net-(R13-Pad2)
- U2 pad 7: Net-(J7-Pad1) -> Net-(J6-Pad2)
Routing:
- net -15V: track 122.2 -> 6.20 mm, vias 10 -> 0
- net +15V: track 76.9 -> 6.20 mm, vias 4 -> 0
- net Net-(R3-Pad2): track 0.00 -> 64.2 mm
- net Net-(J6-Pad2): track 0.00 -> 40.1 mm
- net Net-(J3-Pad3): track 0.00 -> 29.6 mm
- net Net-(J5-Pad2) (its old number): track 27.4 -> 0.00 mm
- net Net-(J6-Pad1): track 25.8 -> 0.00 mm
- net Net-(J3-Pad2): track 0.00 -> 25.7 mm
- net Net-(J7-Pad1): track 25.2 -> 0.00 mm
- net Net-(R4-Pad2): track 0.00 -> 25.1 mm
- net Net-(R2-Pad2): track 0.00 -> 24.7 mm
- net Net-(J6-Pad3): track 0.00 -> 20.4 mm
- net Net-(J1-Pad3): track 18.3 -> 0.00 mm
- net Net-(J2-Pad2) (its old number): track 17.3 -> 0.00 mm
- net GND: track 16.3 -> 0.00 mm, vias 177 -> 0
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- removed copper zone on F.Cu, net GND
Other:
- board size 70 x 54.8 mm -> 100 x 55 mm
- board text added: "Rev 1.0"
- board text removed: "Rev 2.0"

Commit message: finished layout
Parts:
- moved SW2 16.3 mm to (90.0, 110.0), turned to 0 degrees
- moved SW3 16.3 mm to (160.0, 110.0), turned to 180 degrees
- moved J5 13.8 mm to (107.5, 105.0)
- moved J6 13.8 mm to (142.5, 105.0)
- moved R16 6.58 mm to (99.2, 120.8), turned to 90 degrees
- moved R17 5.34 mm to (150.8, 119.5), turned to 90 degrees
- moved R15 5.32 mm to (102.2, 120.8), turned to 90 degrees
- moved SW1 5.00 mm to (125.0, 130.0)
- moved R18 4.59 mm to (147.8, 119.5), turned to 90 degrees
- moved C8 2.51 mm to (151.5, 125.8)
- moved R4 2.51 mm to (151.5, 128.8)
- moved C5 2.50 mm to (81.8, 125.8)
- moved C6 2.50 mm to (98.2, 125.8)
- moved C7 2.50 mm to (168.2, 125.8)
- moved R1 2.50 mm to (81.8, 128.8)
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Connections:
- J5 pad 1: Net-(J5-Pad1) -> GND
- J5 pad 3: GND -> Net-(J5-Pad3)
- J6 pad 1: GND -> Net-(J6-Pad1)
- J6 pad 3: Net-(J6-Pad3) -> GND
- R12 pad 1: Net-(J5-Pad1) -> Net-(J5-Pad3)
- R14 pad 1: Net-(J6-Pad3) -> Net-(J6-Pad1)
- R15 pad 1: Net-(J5-Pad1) -> Net-(R12-Pad2)
- R16 pad 1: Net-(J5-Pad1) -> Net-(R12-Pad2)
- R17 pad 1: Net-(J6-Pad3) -> Net-(R14-Pad2)
- R18 pad 1: Net-(J6-Pad3) -> Net-(R14-Pad2)
- SW2 pad 1: Net-(J5-Pad2) -> Net-(R11-Pad2)
- SW2 pad 2: Net-(J5-Pad2) -> Net-(R11-Pad2)
- SW3 pad 1: Net-(J6-Pad2) -> Net-(R13-Pad2)
- SW3 pad 2: Net-(J6-Pad2) -> Net-(R13-Pad2)
- U1 pad 7: Net-(J5-Pad1) -> Net-(J5-Pad3)
- U2 pad 1: Net-(J6-Pad3) -> Net-(J6-Pad1)
Routing:
- net +15V: track 6.20 -> 115.8 mm, vias 0 -> 4
- net -15V: track 6.20 -> 99.1 mm, vias 0 -> 4
- net Net-(R4-Pad2): track 25.1 -> 69.9 mm
- net Net-(J5-Pad3): track 0.00 -> 33.9 mm
- net Net-(J6-Pad1): track 0.00 -> 32.5 mm
- net Net-(J6-Pad3): track 20.4 -> 0.00 mm
- net Net-(J5-Pad1): track 19.8 -> 0.00 mm
- net GND: track 0.00 -> 14.8 mm, vias 0 -> 169
- net Net-(R13-Pad2): track 7.95 -> 20.8 mm
- net Net-(R11-Pad2): track 8.47 -> 19.9 mm
- net Net-(R12-Pad2): track 0.00 -> 10.1 mm
- net Net-(R16-Pad2): track 6.03 -> 11.2 mm
- net Net-(R15-Pad2): track 9.81 -> 14.9 mm
- net Net-(R18-Pad2): track 9.81 -> 13.8 mm
- net Net-(J3-Pad2): track 25.7 -> 29.7 mm
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- added copper zone on F.Cu, net GND
Other:
- board text added: "16dB"
- board text added: "20dB"
- board text added: "26dB"
- board text added: "28dB"
- board text added: "2CH"
- board text added: "BTL"
- board text added: "CH1 OUT"
- board text added: "CH1/BTL INPUT"
- board text added: "CH2 INPUT"
- board text added: "CH2 OUT"
- board text added: "GAIN"
- board text added: "MODE"
- board text added: "OFF OFF"
- board text added: "OFF ON"
- board text added: "ON OFF"
- board text added: "ON ON"
- board text removed: "1"
- board text removed: "1-2 26dB"
- board text removed: "2"
- board text removed: "2 21dB"
- board text removed: "2-3 29dB"
- board text removed: "3"
